File: herbie2/herbie2_pcb/herbie2.sch (KiCad schematic (older format))
At the start: 6 parts

Commit message: updated PCB
Parts:
- removed B1: ARDUINO_UNO_R3_SHIELD_ICSP-NO_LABELS, Sparkfun_boards:UNO_R3_SHIELD_ICSP_NOLABELS, symbol Sparkfun_boards:ARDUINO_UNO_R3_SHIELD_ICSP-NO_LABELS
- added D1, D2, D3, D4: LED, LED_SMD:LED_1206_3216Metric, symbol Device:LED
- added J1, J2: Screw_Terminal_01x04, TerminalBlock:TerminalBlock_bornier-4_P5.08mm, symbol Connector:Screw_Terminal_01x04
- added J3, J8: I2C_STANDARDQWIIC, Connectors:1X04_1MM_RA, symbol SparkFun-Connectors:I2C_STANDARDQWIIC
- added J4: Servo0, Connector_PinHeader_2.54mm:PinHeader_1x03_P2.54mm_Vertical, symbol Connector:Conn_01x03_Male
- added J5: Servo1, Connector_PinHeader_2.54mm:PinHeader_1x03_P2.54mm_Vertical, symbol Connector:Conn_01x03_Male
- added J6: Servo2, Connector_PinHeader_2.54mm:PinHeader_1x03_P2.54mm_Vertical, symbol Connector:Conn_01x03_Male
- added J7: Servo3, Connector_PinHeader_2.54mm:PinHeader_1x03_P2.54mm_Vertical, symbol Connector:Conn_01x03_Male
- added Q1, Q2: LTC4412ES6_TRMPBF, digikey-footprints:SOT-23-6, symbol dk_PMIC-OR-Controllers-Ideal-Diodes:LTC4412ES6_TRMPBF
- added R1, R2: 470K, Resistor_SMD:R_1206_3216Metric, symbol Device:R
- added R3, R4, R5, R6: R, Resistor_SMD:R_1206_3216Metric, symbol Device:R
Connections:
- net labels added: GND, SERVO_PWR
- wire segments 0 -> 37

Commit message: updated PCB
Parts:
- added F1: Fuse, Fuse:Fuseholder_Blade_Mini_Keystone_3568, symbol Device:Fuse
- added J9: I2C_STANDARDQWIIC, Connectors:1X04_1MM_RA, symbol SparkFun-Connectors:I2C_STANDARDQWIIC
- added LCD1: LCD-16X2SILK, Displays:LCD-16X2, symbol SparkFun-Displays:LCD-16X2SILK
- added U1, U2: 74164, Package_SO:TSSOP-14_4.4x5mm_P0.65mm, symbol 74xx_IEEE:74164
- added U3: 74HC595, Package_SO:SOIC-16_3.9x9.9mm_P1.27mm, symbol 74xx:74HC595
- R3, R4, R5, R6: value R -> 330
Connections:
- net GND: now also B2.GND@ (GND), B2.GND_ (GND), D1.1 (K), D2.1 (K), D3.1 (K), D4.1 (K), J9.1 (GND), LCD1.1 (VSS), LCD1.5 (R/W), U1.7 (Vss), U2.7 (Vss)
- net Vdd: now reaches B2.5V
- net Vdd: now also B2.5V_I (VCC), LCD1.2 (VDD), U1.14 (Vdd), U2.14 (Vdd)
- net ENC1_CS: now reaches B2.D10 (*D10)
- net ENC2_CS: now reaches B2.D11 (*D11)
- net CLK_SERVO: now reaches B2.D12
- net CLK_SERVO: now also U1.8 (CK)
- net DATA_SERVO: now reaches B2.D13
- net DATA_SERVO: now also U1.1 (A), U1.2 (B)
- net CLK_LCD: now reaches B2.D6 (*D6)
- net CLK_LCD: now also U2.8 (CK)
- net DATA_LCD: now reaches B2.D7
- net DATA_LCD: now also U2.1 (A), U2.2 (B)
- net ENC_MISO: now reaches B2.MISO
- net ENC_MOSI: now reaches B2.MOSI
- net ENC_SCK: now reaches B2.SCK
- net at J4.1 (Pin_1): now also U1.6 (Qd)
- net at J5.1 (Pin_1): now also U1.5 (Qc)
- net at J6.1 (Pin_1): now also U1.4 (Qb)
- net at J7.1 (Pin_1): now also U1.3 (Qa)
- net at R3.1: now also U3.3 (QD)
- net at R4.1: now also U3.2 (QC)
- net at R5.1: now also U3.1 (QB)
- net at R6.1: now also U3.15 (QA)
- new net DB4: LCD1.11 (DB4), U2.4 (Qb)
- new net DB5: LCD1.12 (DB5), U2.5 (Qc)
- new net DB6: LCD1.13 (DB6), U2.6 (Qd)
- new net DB7: LCD1.14 (DB7), U2.10 (Qe)
- new net LCD_E: LCD1.6 (E)
- new net LCD_RS: LCD1.4 (RS), U2.3 (Qa)
Other:
- moved on the sheet: D1, D2, D3, D4, J4, J5, J6, J7, R3, R4, R5, R6

Commit message: updated PCB and added footprint library
Parts:
- removed U1: 74164, Package_SO:TSSOP-14_4.4x5mm_P0.65mm, symbol 74xx_IEEE:74164
- removed U3: 74HC595, Package_SO:SOIC-16_3.9x9.9mm_P1.27mm, symbol 74xx:74HC595
- added D5: CVFD20065A, Package_TO_SOT_THT:TO-220-2_Vertical, symbol Diode:CVFD20065A
- added F2: Fuse, Fuse:Fuseholder_Blade_Mini_Keystone_3568, symbol Device:Fuse
- added J10, J11: CONN_04JST-PTH, Connectors:JST-4-PTH, symbol SparkFun-Connectors:CONN_04JST-PTH
- added Q3, Q4: Si4427, js:SO-8_3.9x4.9mm_P1.27mm_Si4427, symbol js:Si4427
- added U1: 74HC595, Package_SO:SOIC-16_3.9x9.9mm_P1.27mm, symbol 74xx:74HC595
- added U3, U7: 24v13_Pololu, js:24v13_Pololu, symbol js:24v13_Pololu
- added U4, U5: LS7366R, Package_SO:SOIC-14_3.9x8.7mm_P1.27mm, symbol js:LS7366R
- added U6: TCA9534, Package_SO:SOIC-16_4.55x10.3mm_P1.27mm, symbol Interface_Expansion:TCA9534
- J1: value Screw_Terminal_01x04 -> GND
- J2: value Screw_Terminal_01x04 -> 5V
- Q1, Q2: value LTC4412ES6_TRMPBF -> LTC4412; symbol dk_PMIC-OR-Controllers-Ideal-Diodes:LTC4412ES6_TRMPBF -> herbie2-rescue:LTC4412ES6_TRMPBF-dk_PMIC-OR-Controllers-Ideal-Diodes
Connections:
- net ENC1_CS is gone; now on net CLK_SERVO: B2.D10 (*D10)
- net ENC2_CS is gone; now on net DATA_SERVO: B2.D11 (*D11)
- net CLK_LCD: now also B2.D3 (*D3); no longer B2.D6 (*D6)
- net CLK_SERVO: now also U1.11 (SRCLK); no longer B2.D12
- net DATA_LCD: now also B2.D4; no longer B2.D7
- net DATA_SERVO: now also U1.14 (SER); no longer B2.D13
- net ENC_MISO: now also U4.6 (miso), U5.6 (miso)
- net ENC_MOSI: now also U4.7 (mosi), U5.7 (mosi)
- net ENC_SCK: now also U4.5 (sck), U5.5 (sck)
- net GND: now also Q1.3 (CTL), Q2.3 (CTL), J10.1, J11.1, U1.13 (~OE), U1.8 (GND), U3.1 (GND), U4.3 (vss), U5.3 (vss), U6.1 (A0), U6.2 (A1), U6.3 (A2), U6.8 (GND), U7.1 (GND); no longer U2.7 (Vss)
- net LCD_E: now also B2.D2
- net Vdd: no longer B2.5V, B2.5V_I (VCC), LCD1.2 (VDD)
- net BATT2: now reaches Q1.1 (VIN)
- net BATT2: now also Q4.3 (D)
- net at Q1.5 (GATE): now also Q4.1 (G)
- net VIN_SW: now reaches Q1.6 (SENSE)
- net VIN_SW: now also Q2.6 (SENSE), R1.2, R2.2, D5.1 (K), Q3.2 (S), Q4.2 (S)
- net VIN_MEASURE: now reaches B2.A3
- net MOT_CURRENT1: now reaches B2.A4
- net MOT_CURRENT2: now reaches B2.A5
- net MOTOR1_DIR: now reaches B2.D5 (*D5)
- net MOTOR1_DIR: now also U3.2 (DIR)
- net MOTOR2_PWM: now reaches B2.D8
- net MOTOR2_PWM: now also U7.3 (PWM)
- net RCLK_SERVO: now reaches B2.D9 (*D9)
- net RCLK_SERVO: now also U1.12 (RCLK)
- net SCL: now reaches B2.SCL
- net SCL: now also J3.4 (SCL), J8.4 (SCL), J9.4 (SCL), U6.14 (SCL)
- net SDA: now reaches B2.SDA
- net SDA: now also J3.3 (SDA), J8.3 (SDA), J9.3 (SDA), U6.15 (SDA)
- net BATT1: now reaches Q2.1 (VIN)
- net BATT1: now also Q3.3 (D)
- net at Q2.5 (GATE): now also Q3.1 (G)
- net 3.3V: now reaches U2.9 (~R)
- net 3.3V: now also J3.2 (VCC), J8.2 (VCC), J9.2 (VCC), J10.2, J11.2, U1.10 (~SRCLR), U1.16 (VCC), U4.14 (vdd), U5.14 (vdd), U6.16 (VDD)
- net at J7.1 (Pin_1): now also U1.15 (QA)
- net at J6.1 (Pin_1): now also U1.1 (QB)
- net at J5.1 (Pin_1): now also U1.2 (QC)
- net at J4.1 (Pin_1): now also U1.3 (QD)
- net at R3.1: now also U6.7 (P3)
- net at R4.1: now also U6.6 (P2)
- net at R5.1: now also U6.5 (P1)
- net at R6.1: now also U6.4 (P0)
- new net: J11.4, U4.11 (b)
- new net: J11.3, U4.12 (a)
- new net: J10.4, U5.11 (b)
- new net: J10.3, U5.12 (a)
- new net 5V: B2.5V, B2.5V_I (VCC), LCD1.2 (VDD)
- new net AC_PWR: D5.2 (A)
- new net ENC1_SS: B2.D12, U4.4 (ss)
- new net ENC2_SS: B2.D13, U5.4 (ss)
- new net MOTOR1_PWM: B2.D6 (*D6), U3.3 (PWM)
- new net MOTOR2_DIR: B2.D7, U7.2 (DIR)
- new net Vss: U2.7 (Vss)
Other:
- moved on the sheet: F1, Q1, Q2, R1, R2

Commit message: updated PCB
Parts:
- added C1, C2, C3, C4: 12pF, Capacitor_SMD:C_1206_3216Metric, symbol pspice:C
- added C5, C6, C7, C8: .1uF, Capacitor_SMD:C_1206_3216Metric, symbol Device:C
- added H10: AC_PWR, MountingHole:MountingHole_2.2mm_M2_Pad, symbol Mechanical:MountingHole_Pad
- added H5: GND_BATT1, MountingHole:MountingHole_2.2mm_M2_Pad, symbol Mechanical:MountingHole_Pad
- added H6: PWR_BATT1, MountingHole:MountingHole_2.2mm_M2_Pad, symbol Mechanical:MountingHole_Pad
- added H7: GND_BATT2, MountingHole:MountingHole_2.2mm_M2_Pad, symbol Mechanical:MountingHole_Pad
- added H8: PWR_BATT2, MountingHole:MountingHole_2.2mm_M2_Pad, symbol Mechanical:MountingHole_Pad
- added H9: GND_AC_PWR, MountingHole:MountingHole_2.2mm_M2_Pad, symbol Mechanical:MountingHole_Pad
- added J12: Vin, TerminalBlock:TerminalBlock_bornier-4_P5.08mm, symbol Connector:Screw_Terminal_01x04
- added J13: Servo4, Connector_PinHeader_2.54mm:PinHeader_1x03_P2.54mm_Vertical, symbol Connector:Conn_01x03_Male
- added J14: Servo5, Connector_PinHeader_2.54mm:PinHeader_1x03_P2.54mm_Vertical, symbol Connector:Conn_01x03_Male
- added J15: Conn_01x03_Male, Connector_PinHeader_2.54mm:PinHeader_1x03_P2.54mm_Vertical, symbol Connector:Conn_01x03_Male
- added J16: Conn_02x04_Odd_Even, Connector_PinHeader_2.54mm:PinHeader_2x04_P2.54mm_Vertical, symbol Connector_Generic:Conn_02x04_Odd_Even
- added R10, R11, R12, R9: 100, Resistor_SMD:R_1206_3216Metric, symbol Device:R
- added R13: 10, Resistor_SMD:R_1206_3216Metric, symbol Device:R
- added R14, R15, R16, R17: 20K, Resistor_SMD:R_1206_3216Metric, symbol Device:R
- added R18, R19: 1M, Resistor_SMD:R_1206_3216Metric, symbol Device:R
- added R7, R8: R, Resistor_SMD:R_1206_3216Metric, symbol Device:R
- added U8: D36V50F5_Pololu, js:D36V50F5_Pololu, symbol js:D36V50F5_Pololu
- added Y1, Y2: 20MHz, Crystal:Crystal_SMD_5032-2Pin_5.0x3.2mm_HandSoldering, symbol Device:Crystal
- J4: value Servo0 -> Servo3
- J5: value Servo1 -> Servo2
- J6: value Servo2 -> Servo1
- J7: value Servo3 -> Servo0
Connections:
- net 3.3V: now also C5.2, C6.2, C7.1, C8.1, R14.1, R15.1, R16.1, R17.1
- net 5V: now also J2.1 (Pin_1), J2.2 (Pin_2), J2.3 (Pin_3), J2.4 (Pin_4), R13.1, U8.1 (Vout); no longer B2.5V
- net GND: now also J1.1 (Pin_1), J1.2 (Pin_2), J1.3 (Pin_3), J1.4 (Pin_4), LCD1.16 (K), C1.2, C2.2, C3.2, C4.2, C5.1, C6.1, C7.2, C8.2, J13.3 (Pin_3), J14.3 (Pin_3), J15.3 (Pin_3), J16.2 (Pin_2), J16.4 (Pin_4), J16.6 (Pin_6), J16.8 (Pin_8), R8.2, U8.2 (GND)
- net SERVO_PWR: now also J13.2 (Pin_2), J14.2 (Pin_2)
- net VIN_MEASURE: now also R7.2, R8.1
- net VIN_SW: now also J12.1 (Pin_1), J12.2 (Pin_2), J12.3 (Pin_3), J12.4 (Pin_4), R7.1, U8.3 (Vin)
- net at U4.1 (fcko): now also C4.1, R19.1, Y2.2
- net at U4.11 (b): now also R10.2; no longer J11.4
- net at U4.12 (a): now also R9.2; no longer J11.3
- net at U4.2 (fcki): now also C3.1, R19.2, Y2.1
- net at U5.1 (fcko): now also C1.1, R18.2, Y1.1
- net at U5.11 (b): now also R12.2; no longer J10.4
- net at U5.12 (a): now also R11.2; no longer J10.3
- net at U5.2 (fcki): now also C2.1, R18.1, Y1.2
- net at LCD1.15 (A): now also R13.2
- net DI1: now reaches U6.10 (P5)
- net DI1: now also J16.3 (Pin_3)
- net DI2: now reaches U6.11 (P6)
- net DI2: now also J16.5 (Pin_5)
- net DI3: now reaches U6.12 (P7)
- net DI3: now also J16.7 (Pin_7)
- net DI0: now reaches U6.9 (P4)
- net DI0: now also J16.1 (Pin_1)
- net E_STOP1: now reaches U3.4 (/SLP)
- net E_STOP1: now also J15.1 (Pin_1)
- net E_STOP2: now reaches U7.4 (/SLP)
- net E_STOP2: now also J15.2 (Pin_2)
- net at U1.4 (QE): now also J13.1 (Pin_1)
- net at U1.5 (QF): now also J14.1 (Pin_1)
- new net: J10.3, R11.1, R16.2
- new net: J10.4, R12.1, R14.2
- new net: J11.3, R17.2, R9.1
- new net: J11.4, R10.1, R15.2
- new net 5V_USB: B2.5V
Other:
- moved on the sheet: D5, J1, J10, J11, J2, U4, U5, U6

Commit message: started routing board
Parts:
- removed J16: Conn_02x04_Odd_Even, Connector_PinHeader_2.54mm:PinHeader_2x04_P2.54mm_Vertical, symbol Connector_Generic:Conn_02x04_Odd_Even
- added J16: Conn_02x03_Odd_Even, Connector_PinHeader_2.54mm:PinHeader_2x03_P2.54mm_Vertical, symbol Connector_Generic:Conn_02x03_Odd_Even
- added Q5: 2N7002, digikey-footprints:SOT-23-3, symbol dk_Transistors-FETs-MOSFETs-Single:2N7002
- added R20: 1K, Resistor_SMD:R_1206_3216Metric, symbol Device:R
- added RV1: 1K, Potentiometer_THT:Potentiometer_Bourns_3266Y_Vertical, symbol Device:R_POT
Connections:
- net labels added: BATT1_F, LCD_BL, VIN, VIN_FUSE
- net labels removed: DI3, VIN_SW
- wire segments 288 -> 311
Other:
- moved on the sheet: F1
Changed lines of the file:
@@
 L Device:Fuse F1
 U 1 1 5FD09C9A
-P 700 1900
-F 0 "F1" H 760 1946 50  0000 L CNN
-F 1 "Fuse" H 760 1855 50  0000 L CNN
-F 2 "Fuse:Fuseholder_Blade_Mini_Keystone_3568" V 630 1900 50  0001 C CNN
-F 3 "~" H 700 1900 50  0001 C CNN
-	1    700  1900
+P 2000 2750
+F 0 "F1" H 2060 2796 50  0000 L CNN
+F 1 "Fuse" H 2060 2705 50  0000 L CNN
+F 2 "Fuse:Fuseholder_Blade_Mini_Keystone_3568" V 1930 2750 50  0001 C CNN
+F 3 "~" H 2000 2750 50  0001 C CNN
+	1    2000 2750
 	1    0    0    -1
 $EndComp
@@
 Wire Wire Line
 	3700 2950 3700 3100
-Text GLabel 3300 2800 1    50   Input ~ 0
-BATT1
 Wire Wire Line
 	3400 3550 3350 3550
@@
 Wire Wire Line
 	2400 4450 2900 4450
-Text GLabel 2650 2900 2    50   Input ~ 0
-VIN_SW
 Text GLabel 2600 4150 2    50   Input ~ 0
-VIN_SW
+VIN_FUSE
 Text GLabel 2850 3300 0    50   Input ~ 0
-VIN_SW
+VIN_FUSE
 Text GLabel 2850 4550 0    50   Input ~ 0
-VIN_SW
+VIN_FUSE
 Wire Wire Line
 	2850 4550 2900 4550
@@
 Wire Wire Line
 	2650 2900 2550 2900
-Text GLabel 2100 2900 0    50   Input ~ 0
+Text GLabel 2000 2550 0    50   Input ~ 0
 BATT1
 Text GLabel 2050 4150 0    50   Input ~ 0
 BATT2
 Wire Wire Line
-	2100 2900 2150 2900
-Wire Wire Line
 	2050 4150 2100 4150
 Text GLabel 3750 2650 2    50   Input ~ 0
-VIN_SW
+VIN_FUSE
 Text GLabel 3750 3900 2    50   Input ~ 0
-VIN_SW
+VIN_FUSE
 Wire Wire Line
 	3750 3900 3700 3900
@@
 	3350 2100 3450 2100
 Text GLabel 3900 2100 2    50   Input ~ 0
-VIN_SW
+VIN_FUSE
 Wire Wire Line
 	3900 2100 3750 2100
@@
 GND
 Text GLabel 5050 1100 0    50   Input ~ 0
-VIN_SW
+VIN
 Text GLabel 5050 900  0    50   Input ~ 0
 5V
@@
 GND
 Text GLabel 4750 2400 0    50   Input ~ 0
-VIN_SW
+VIN
 Wire Wire Line
 	4750 2400 4800 2400
@@
 Wire Wire Line
 	9550 3250 10150 3250
-Text GLabel 9750 3350 0    50   Input ~ 0
+Text GLabel 9700 3800 0    50   Input ~ 0
 GND
 Wire Wire Line
@@
 GND
 Text GLabel 1000 2500 0    50   Input ~ 0
-VIN_SW
+VIN
 Wire Wire Line
 	1000 2500 1100 2500
@@
 DI2
 Text GLabel 6800 5750 2    50   Input ~ 0
-DI3
+LCD_BL
 Wire Wire Line
 	6550 5450 6800 5450
@@
 Wire Wire Line
 	6550 5750 6800 5750
-$Comp
-L Connector_Generic:Conn_02x04_Odd_Even J16
-U 1 1 60CDD4DB
-P 4750 5050
-F 0 "J16" H 4800 5367 50  0000 C CNN
-F 1 "Conn_02x04_Odd_Even" H 4800 5276 50  0000 C CNN
-F 2 "Connector_PinHeader_2.54mm:PinHeader_2x04_P2.54mm_Vertical" H 4750 5050 50  0001 C CNN
-F 3 "~" H 4750 5050 50  0001 C CNN
-	1    4750 5050
-	1    0    0    -1
-$EndComp
 Text GLabel 5150 4950 2    50   Input ~ 0
 GND
 Wire Wire Line
 	5150 4950 5050 4950
-Wire Wire Line
-	5050 5050 5050 4950
-Connection ~ 5050 4950
-Wire Wire Line
-	5050 5150 5050 5050
-Connection ~ 5050 5050
-Wire Wire Line
-	5050 5250 5050 5150
-Connection ~ 5050 5150
 Text GLabel 4400 4950 0    50   Input ~ 0
 DI0
@@
 Text GLabel 4400 5150 0    50   Input ~ 0
 DI2
-Text GLabel 4400 5250 0    50   Input ~ 0
-DI3
 Wire Wire Line
 	4400 4950 4550 4950
@@
 Wire Wire Line
 	4400 5150 4550 5150
-Wire Wire Line
-	4400 5250 4550 5250
+Text GLabel 9100 700  2    50   Input ~ 0
+3.3V
+Wire Wire Line
+	9100 700  9050 700
+Wire Wire Line
+	9050 700  9050 800
+Text GLabel 8550 750  0    50   Input ~ 0
+GND
+Wire Wire Line
+	8550 750  8850 750
+Wire Wire Line
+	8850 750  8850 800
+$Comp
+L dk_Transistors-FETs-MOSFETs-Single:2N7002 Q5
+U 1 1 5FDB34D9
+P 9750 3550
+F 0 "Q5" H 9858 3603 60  0000 L CNN
+F 1 "2N7002" H 9858 3497 60  0000 L CNN
+F 2 "digikey-footprints:SOT-23-3" H 9950 3750 60  0001 L CNN
+F 3 "https://www.onsemi.com/pub/Collateral/NDS7002A-D.PDF" H 9950 3850 60  0001 L CNN
+F 4 "2N7002NCT-ND" H 9950 3950 60  0001 L CNN "Digi-Key_PN"
+F 5 "2N7002" H 9950 4050 60  0001 L CNN "MPN"
+F 6 "Discrete Semiconductor Products" H 9950 4150 60  0001 L CNN "Category"
+F 7 "Transistors - FETs, MOSFETs - Single" H 9950 4250 60  0001 L CNN "Family"
+F 8 "https://www.onsemi.com/pub/Collateral/NDS7002A-D.PDF" H 9950 4350 60  0001 L CNN "DK_Datasheet_Link"
+F 9 "/product-detail/en/on-semiconductor/2N7002/2N7002NCT-ND/244664" H 9950 4450 60  0001 L CNN "DK_Detail_Page"
+F 10 "MOSFET N-CH 60V 115MA SOT-23" H 9950 4550 60  0001 L CNN "Description"
+F 11 "ON Semiconductor" H 9950 4650 60  0001 L CNN "Manufacturer"
+F 12 "Active" H 9950 4750 60  0001 L CNN "Status"
+	1    9750 3550
+	1    0    0    -1
+$EndComp
+Wire Wire Line
+	9700 3800 9750 3800
+Wire Wire Line
+	9750 3800 9750 3750
+$Comp
+L Device:R R20
+U 1 1 5FED41B4
+P 9250 3650
+F 0 "R20" H 9320 3696 50  0000 L CNN
+F 1 "1K" H 9320 3605 50  0000 L CNN
+F 2 "Resistor_SMD:R_1206_3216Metric" V 9180 3650 50  0001 C CNN
+F 3 "~" H 9250 3650 50  0001 C CNN
+	1    9250 3650
+	0    1    1    0
+$EndComp
+Wire Wire Line
+	9400 3650 9450 3650
+Text GLabel 9000 3650 0    50   Input ~ 0
+LCD_BL
+Wire Wire Line
+	9000 3650 9100 3650
+$Comp
+L Connector_Generic:Conn_02x03_Odd_Even J16
+U 1 1 5FF45C1B
+P 4750 5050
+F 0 "J16" H 4800 5367 50  0000 C CNN
+F 1 "Conn_02x03_Odd_Even" H 4800 5276 50  0000 C CNN
+F 2 "Connector_PinHeader_2.54mm:PinHeader_2x03_P2.54mm_Vertical" H 4750 5050 50  0001 C CNN
+F 3 "~" H 4750 5050 50  0001 C CNN
+	1    4750 5050
+	1    0    0    -1
+$EndComp
+Wire Wire Line
+	5050 5150 5050 5050
+Wire Wire Line
+	5050 5050 5050 4950
+Connection ~ 5050 5050
+Connection ~ 5050 4950
+Text GLabel 900  1750 0    50   Input ~ 0
+VIN
+Text GLabel 900  2050 0    50   Input ~ 0
+VIN_FUSE
+Wire Wire Line
+	900  1750 1000 1750
+Wire Wire Line
+	900  2050 1000 2050
+Text GLabel 2650 2800 2    50   Input ~ 0
+VIN_FUSE
+Wire Wire Line
+	2650 2800 2650 2900
+Text GLabel 1950 2200 2    50   Input ~ 0
+AC_PWR
+Text GLabel 1950 1900 2    50   Input ~ 0
+GND
+Text GLabel 1950 1650 2    50   Input ~ 0
+BATT2
+Text GLabel 1950 1400 2    50   Input ~ 0
+GND
+Text GLabel 1950 1100 2    50   Input ~ 0
+BATT1
+Text GLabel 1950 850  2    50   Input ~ 0
+GND
+Wire Wire Line
+	1550 850  1950 850
+Wire Wire Line
+	1550 1100 1950 1100
+Wire Wire Line
+	1550 1400 1950 1400
+Wire Wire Line
+	1550 1650 1950 1650
+Wire Wire Line
+	1550 1900 1950 1900
+Wire Wire Line
+	1550 2200 1950 2200
+$Comp
+L Device:R_POT RV1
+U 1 1 602D06E5
+P 9250 2400
+F 0 "RV1" H 9180 2446 50  0000 R CNN
+F 1 "1K" H 9180 2355 50  0000 R CNN
+F 2 "Potentiometer_THT:Potentiometer_Bourns_3266Y_Vertical" H 9250 2400 50  0001 C CNN
+F 3 "~" H 9250 2400 50  0001 C CNN
+	1    9250 2400
+	1    0    0    -1
+$EndComp
+Text GLabel 9150 2250 0    50   Input ~ 0
+5V
+Text GLabel 9150 2550 0    50   Input ~ 0
+GND
+Wire Wire Line
+	9150 2250 9250 2250
+Wire Wire Line
+	9150 2550 9250 2550
+Wire Wire Line
+	9400 2400 9400 2050
+Wire Wire Line
+	9400 2050 10150 2050
+Wire Wire Line
+	2000 2900 2050 2900
+Text GLabel 2050 3000 0    50   Input ~ 0
+BATT1_F
+Wire Wire Line
+	2050 3000 2050 2900
+Connection ~ 2050 2900
+Wire Wire Line
+	2050 2900 2150 2900
+Text GLabel 3300 2800 1    50   Input ~ 0
+BATT1_F
+Wire Wire Line
+	2000 2550 2000 2600
+Text GLabel 6150 3050 0    50   Input ~ 0
+3.3V
+Wire Wire Line
+	6150 3050 6350 3050
 $EndSCHEMATC

Commit message: routed board
Parts:
- added H11, H12, H13: MountingHole_Pad, MountingHole:MountingHole_2.2mm_M2_Pad_TopBottom, symbol Mechanical:MountingHole_Pad
- added J17, J20: Conn_01x03, Connector_PinHeader_2.54mm:PinHeader_1x03_P2.54mm_Vertical, symbol Connector_Generic:Conn_01x03
- added J18, J5: Conn_01x02, Connector_PinHeader_2.54mm:PinHeader_1x02_P2.54mm_Vertical, symbol Connector_Generic:Conn_01x02
- added J19, J4: Conn_01x01, Connector_PinHeader_2.54mm:PinHeader_1x01_P2.54mm_Vertical, symbol Connector_Generic:Conn_01x01
- added R21, R22: 47K, Resistor_SMD:R_1206_3216Metric, symbol Device:R
- renumbered J7 to S0, J6 to S1, J5 to S2, J4 to S3, J13 to S4, J14 to S5
Connections:
- net labels added: 5V_REG
- net labels removed: 5V_USB, MOT_CURRENT1, MOT_CURRENT2, SERVO_PWR
- wire segments 311 -> 347
- no-connect marks 0 -> 20

Commit message: changed PWM pins
Parts:
- added C10: 1uF, Capacitor_SMD:C_1206_3216Metric, symbol Device:C
- added C11: 10uF, Capacitor_SMD:C_1206_3216Metric, symbol Device:C
- added C9: .1uF, Capacitor_SMD:C_1206_3216Metric, symbol Device:C
Connections:
- wire segments 347 -> 353
Changed lines of the file:
@@
 Wire Wire Line
 	1200 5300 1300 5300
-Text GLabel 7550 2850 2    50   Input ~ 0
+Text GLabel 7550 3050 2    50   Input ~ 0
 MOTOR1_DIR
 Text GLabel 7550 3150 2    50   Input ~ 0
 MOTOR2_DIR
-Text GLabel 7550 2950 2    50   Input ~ 0
-MOTOR1_PWM
-Text GLabel 7550 3050 2    50   Input ~ 0
-MOTOR2_PWM
 Wire Wire Line
 	7350 2550 7550 2550
@@
 Wire Wire Line
 	6600 1100 6700 1100
+$Comp
+L Device:C C11
+U 1 1 5FD6E330
+P 5850 6600
+F 0 "C11" H 5965 6646 50  0000 L CNN
+F 1 "10uF" H 5965 6555 50  0000 L CNN
+F 2 "Capacitor_SMD:C_1206_3216Metric" H 5888 6450 50  0001 C CNN
+F 3 "~" H 5850 6600 50  0001 C CNN
+	1    5850 6600
+	1    0    0    -1
+$EndComp
+$Comp
+L Device:C C10
+U 1 1 5FD6E6D3
+P 5550 6600
+F 0 "C10" H 5665 6646 50  0000 L CNN
+F 1 "1uF" H 5665 6555 50  0000 L CNN
+F 2 "Capacitor_SMD:C_1206_3216Metric" H 5588 6450 50  0001 C CNN
+F 3 "~" H 5550 6600 50  0001 C CNN
+	1    5550 6600
+	1    0    0    -1
+$EndComp
+$Comp
+L Device:C C9
+U 1 1 5FD6EB16
+P 5300 6600
+F 0 "C9" H 5415 6646 50  0000 L CNN
+F 1 ".1uF" H 5415 6555 50  0000 L CNN
+F 2 "Capacitor_SMD:C_1206_3216Metric" H 5338 6450 50  0001 C CNN
+F 3 "~" H 5300 6600 50  0001 C CNN
+	1    5300 6600
+	1    0    0    -1
+$EndComp
+Text GLabel 5550 6900 3    50   Input ~ 0
+GND
+Wire Wire Line
+	5550 6900 5550 6750
+Wire Wire Line
+	5550 6750 5850 6750
+Connection ~ 5550 6750
+Wire Wire Line
+	5550 6750 5300 6750
+Wire Wire Line
+	5300 6450 5550 6450
+Wire Wire Line
+	5850 6450 5550 6450
+Connection ~ 5550 6450
+Text GLabel 5550 6350 1    50   Input ~ 0
+VIN_FUSE
+Wire Wire Line
+	5550 6350 5550 6450
+Text GLabel 7550 2950 2    50   Input ~ 0
+MOTOR2_PWM
+Text GLabel 7550 2850 2    50   Input ~ 0
+MOTOR1_PWM
 $EndSCHEMATC
