File: herbie2/herbie2_pcb/herbie2.sch (KiCad schematic (older format))
At the start: 93 parts, among them J1 GND, J10 CONN_04JST-PTH, J11 CONN_04JST-PTH, J12 Vin, J15 Conn_01x03_Male, J16 Conn_02x03_Odd_Even, J17 Conn_01x03, J18 Conn_01x02, J19 Conn_01x01, J2 5V, J20 Conn_01x03, J3 I2C_STANDARDQWIIC, J4 Conn_01x01, J5 Conn_01x02, J8 I2C_STANDARDQWIIC, J9 I2C_STANDARDQWIIC, Q1 LTC4412, Q2 LTC4412, Q3 Si4427, Q4 Si4427, Q5 2N7002, U1 74HC595, U2 74164, U3 24v13_Pololu, U4 LS7366R, U5 LS7366R, U6 TCA9534, U7 24v13_Pololu, U8 D36V50F5_Pololu, Y1 20MHz, Y2 20MHz

Commit message: added i2c pullup resistors
Parts:
- added C12: 10uF, Capacitor_SMD:C_1206_3216Metric, symbol Device:C
- added R23, R24: R, Resistor_SMD:R_1206_3216Metric, symbol Device:R
Connections:
- wire segments 353 -> 359
Other:
- moved on the sheet: C10, C11, C7, C8, C9
Changed lines of the file:
@@
 L Device:C C7
 U 1 1 60880978
-P 6250 6600
-F 0 "C7" H 6365 6646 50  0000 L CNN
-F 1 ".1uF" H 6365 6555 50  0000 L CNN
-F 2 "Capacitor_SMD:C_1206_3216Metric" H 6288 6450 50  0001 C CNN
-F 3 "~" H 6250 6600 50  0001 C CNN
-	1    6250 6600
-	1    0    0    -1
-$EndComp
-Text GLabel 6250 6900 3    50   Input ~ 0
-GND
-Wire Wire Line
-	6250 6900 6250 6750
+P 6350 6600
+F 0 "C7" H 6465 6646 50  0000 L CNN
+F 1 ".1uF" H 6465 6555 50  0000 L CNN
+F 2 "Capacitor_SMD:C_1206_3216Metric" H 6388 6450 50  0001 C CNN
+F 3 "~" H 6350 6600 50  0001 C CNN
+	1    6350 6600
+	1    0    0    -1
+$EndComp
+Text GLabel 6350 6900 3    50   Input ~ 0
+GND
+Wire Wire Line
+	6350 6900 6350 6750
 $Comp
 L Device:C C8
 U 1 1 6093E7F6
-P 6550 6600
-F 0 "C8" H 6665 6646 50  0000 L CNN
-F 1 ".1uF" H 6665 6555 50  0000 L CNN
-F 2 "Capacitor_SMD:C_1206_3216Metric" H 6588 6450 50  0001 C CNN
-F 3 "~" H 6550 6600 50  0001 C CNN
-	1    6550 6600
+P 6650 6600
+F 0 "C8" H 6765 6646 50  0000 L CNN
+F 1 ".1uF" H 6765 6555 50  0000 L CNN
+F 2 "Capacitor_SMD:C_1206_3216Metric" H 6688 6450 50  0001 C CNN
+F 3 "~" H 6650 6600 50  0001 C CNN
+	1    6650 6600
 	1    0    0    -1
 $EndComp
@@
 	5900 4750 6150 4750
 Wire Wire Line
-	6550 6450 6250 6450
-Wire Wire Line
-	6550 6750 6250 6750
-Connection ~ 6250 6750
-Text GLabel 6650 6400 2    50   Input ~ 0
+	6650 6450 6350 6450
+Wire Wire Line
+	6650 6750 6350 6750
+Connection ~ 6350 6750
+Text GLabel 6750 6400 2    50   Input ~ 0
 3.3V
 Wire Wire Line
-	6650 6400 6550 6400
-Wire Wire Line
-	6550 6400 6550 6450
-Connection ~ 6550 6450
+	6750 6400 6650 6400
+Wire Wire Line
+	6650 6400 6650 6450
+Connection ~ 6650 6450
 Text GLabel 4250 700  2    50   Input ~ 0
 E_STOP1
@@
 L Device:C C11
 U 1 1 5FD6E330
-P 5850 6600
-F 0 "C11" H 5965 6646 50  0000 L CNN
-F 1 "10uF" H 5965 6555 50  0000 L CNN
-F 2 "Capacitor_SMD:C_1206_3216Metric" H 5888 6450 50  0001 C CNN
-F 3 "~" H 5850 6600 50  0001 C CNN
-	1    5850 6600
+P 5650 6550
+F 0 "C11" H 5765 6596 50  0000 L CNN
+F 1 "10uF" H 5765 6505 50  0000 L CNN
+F 2 "Capacitor_SMD:C_1206_3216Metric" H 5688 6400 50  0001 C CNN
+F 3 "~" H 5650 6550 50  0001 C CNN
+	1    5650 6550
 	1    0    0    -1
 $EndComp
@@
 L Device:C C10
 U 1 1 5FD6E6D3
-P 5550 6600
-F 0 "C10" H 5665 6646 50  0000 L CNN
-F 1 "1uF" H 5665 6555 50  0000 L CNN
-F 2 "Capacitor_SMD:C_1206_3216Metric" H 5588 6450 50  0001 C CNN
-F 3 "~" H 5550 6600 50  0001 C CNN
-	1    5550 6600
+P 5350 6550
+F 0 "C10" H 5465 6596 50  0000 L CNN
+F 1 "1uF" H 5465 6505 50  0000 L CNN
+F 2 "Capacitor_SMD:C_1206_3216Metric" H 5388 6400 50  0001 C CNN
+F 3 "~" H 5350 6550 50  0001 C CNN
+	1    5350 6550
 	1    0    0    -1
 $EndComp
@@
 L Device:C C9
 U 1 1 5FD6EB16
-P 5300 6600
-F 0 "C9" H 5415 6646 50  0000 L CNN
-F 1 ".1uF" H 5415 6555 50  0000 L CNN
-F 2 "Capacitor_SMD:C_1206_3216Metric" H 5338 6450 50  0001 C CNN
-F 3 "~" H 5300 6600 50  0001 C CNN
-	1    5300 6600
-	1    0    0    -1
-$EndComp
-Text GLabel 5550 6900 3    50   Input ~ 0
-GND
-Wire Wire Line
-	5550 6900 5550 6750
-Wire Wire Line
-	5550 6750 5850 6750
-Connection ~ 5550 6750
-Wire Wire Line
-	5550 6750 5300 6750
-Wire Wire Line
-	5300 6450 5550 6450
-Wire Wire Line
-	5850 6450 5550 6450
-Connection ~ 5550 6450
-Text GLabel 5550 6350 1    50   Input ~ 0
+P 5100 6550
+F 0 "C9" H 5215 6596 50  0000 L CNN
+F 1 ".1uF" H 5215 6505 50  0000 L CNN
+F 2 "Capacitor_SMD:C_1206_3216Metric" H 5138 6400 50  0001 C CNN
+F 3 "~" H 5100 6550 50  0001 C CNN
+	1    5100 6550
+	1    0    0    -1
+$EndComp
+Text GLabel 5350 6850 3    50   Input ~ 0
+GND
+Wire Wire Line
+	5350 6850 5350 6700
+Wire Wire Line
+	5350 6700 5650 6700
+Connection ~ 5350 6700
+Wire Wire Line
+	5350 6700 5100 6700
+Wire Wire Line
+	5100 6400 5350 6400
+Wire Wire Line
+	5650 6400 5350 6400
+Connection ~ 5350 6400
+Text GLabel 5350 6300 1    50   Input ~ 0
 VIN_FUSE
 Wire Wire Line
-	5550 6350 5550 6450
+	5350 6300 5350 6400
 Text GLabel 7550 2950 2    50   Input ~ 0
 MOTOR2_PWM
 Text GLabel 7550 2850 2    50   Input ~ 0
 MOTOR1_PWM
+$Comp
+L Device:R R23
+U 1 1 5FD8C634
+P 6600 4600
+F 0 "R23" H 6670 4646 50  0000 L CNN
+F 1 "R" H 6670 4555 50  0000 L CNN
+F 2 "Resistor_SMD:R_1206_3216Metric" V 6530 4600 50  0001 C CNN
+F 3 "~" H 6600 4600 50  0001 C CNN
+	1    6600 4600
+	1    0    0    -1
+$EndComp
+$Comp
+L Device:R R24
+U 1 1 5FD8D066
+P 6850 4600
+F 0 "R24" H 6920 4646 50  0000 L CNN
+F 1 "R" H 6920 4555 50  0000 L CNN
+F 2 "Resistor_SMD:R_1206_3216Metric" V 6780 4600 50  0001 C CNN
+F 3 "~" H 6850 4600 50  0001 C CNN
+	1    6850 4600
+	1    0    0    -1
+$EndComp
+Text GLabel 6550 4750 0    50   Input ~ 0
+SCL
+Text GLabel 6900 4750 2    50   Input ~ 0
+SDA
+Text GLabel 6550 4450 0    50   Input ~ 0
+3.3V
+Wire Wire Line
+	6550 4450 6600 4450
+Wire Wire Line
+	6600 4450 6850 4450
+Connection ~ 6600 4450
+Wire Wire Line
+	6550 4750 6600 4750
+Wire Wire Line
+	6900 4750 6850 4750
+$Comp
+L Device:C C12
+U 1 1 5FEEF910
+P 5950 6550
+F 0 "C12" H 6065 6596 50  0000 L CNN
+F 1 "10uF" H 6065 6505 50  0000 L CNN
+F 2 "Capacitor_SMD:C_1206_3216Metric" H 5988 6400 50  0001 C CNN
+F 3 "~" H 5950 6550 50  0001 C CNN
+	1    5950 6550
+	1    0    0    -1
+$EndComp
+Wire Wire Line
+	5950 6400 5650 6400
+Connection ~ 5650 6400
+Wire Wire Line
+	5950 6700 5650 6700
+Connection ~ 5650 6700
 $EndSCHEMATC
