File: herbie2/herbie2_pcb/herbie2.sch (KiCad schematic (older format))
At the start: 96 parts, among them J1 GND, J10 CONN_04JST-PTH, J11 CONN_04JST-PTH, J12 Vin, J15 Conn_01x03_Male, J16 Conn_02x03_Odd_Even, J17 Conn_01x03, J18 Conn_01x02, J19 Conn_01x01, J2 5V, J20 Conn_01x03, J3 I2C_STANDARDQWIIC, J4 Conn_01x01, J5 Conn_01x02, J8 I2C_STANDARDQWIIC, J9 I2C_STANDARDQWIIC, Q1 LTC4412, Q2 LTC4412, Q3 Si4427, Q4 Si4427, Q5 2N7002, U1 74HC595, U2 74164, U3 24v13_Pololu, U4 LS7366R, U5 LS7366R, U6 TCA9534, U7 24v13_Pololu, U8 D36V50F5_Pololu, Y1 20MHz, Y2 20MHz

Commit message: v0.1
Parts:
- added C13: .1uF, Capacitor_SMD:C_1206_3216Metric, symbol Device:C
- R21, R22: value 47K -> 20K
- R23, R24: value R -> 4.7K
- RV1: value 1K -> 10K
Connections:
- wire segments 359 -> 364
Other:
- moved on the sheet: D1, D2, D3, D4
Changed lines of the file:
@@
 F 3 "~" H 7900 6100 50  0001 C CNN
 	1    7900 6100
-	-1   0    0    1
+	1    0    0    -1
 $EndComp
 $Comp
@@
 F 3 "~" H 7900 5750 50  0001 C CNN
 	1    7900 5750
-	-1   0    0    1
+	1    0    0    -1
 $EndComp
 $Comp
@@
 F 3 "~" H 7900 5400 50  0001 C CNN
 	1    7900 5400
-	-1   0    0    1
+	1    0    0    -1
 $EndComp
 $Comp
@@
 F 3 "~" H 7900 5050 50  0001 C CNN
 	1    7900 5050
-	-1   0    0    1
+	1    0    0    -1
 $EndComp
 $Comp
@@
 DATA_LCD
 Text GLabel 8250 5450 2    50   Input ~ 0
-GND
+3.3V
 Wire Wire Line
 	8050 5050 8200 5050
@@
 	6650 6450 6350 6450
 Wire Wire Line
-	6650 6750 6350 6750
+	6650 6750 6500 6750
 Connection ~ 6350 6750
 Text GLabel 6750 6400 2    50   Input ~ 0
@@
 P 9250 2400
 F 0 "RV1" H 9180 2446 50  0000 R CNN
-F 1 "1K" H 9180 2355 50  0000 R CNN
+F 1 "10K" H 9180 2355 50  0000 R CNN
 F 2 "Potentiometer_THT:Potentiometer_Bourns_3266Y_Vertical" H 9250 2400 50  0001 C CNN
 F 3 "~" H 9250 2400 50  0001 C CNN
@@
 P 8250 3500
 F 0 "R22" H 8320 3546 50  0000 L CNN
-F 1 "47K" H 8320 3455 50  0000 L CNN
+F 1 "20K" H 8320 3455 50  0000 L CNN
 F 2 "Resistor_SMD:R_1206_3216Metric" V 8180 3500 50  0001 C CNN
 F 3 "~" H 8250 3500 50  0001 C CNN
@@
 P 8250 3100
 F 0 "R21" H 8320 3146 50  0000 L CNN
-F 1 "47K" H 8320 3055 50  0000 L CNN
+F 1 "20K" H 8320 3055 50  0000 L CNN
 F 2 "Resistor_SMD:R_1206_3216Metric" V 8180 3100 50  0001 C CNN
 F 3 "~" H 8250 3100 50  0001 C CNN
@@
 P 6600 4600
 F 0 "R23" H 6670 4646 50  0000 L CNN
-F 1 "R" H 6670 4555 50  0000 L CNN
+F 1 "4.7K" H 6670 4555 50  0000 L CNN
 F 2 "Resistor_SMD:R_1206_3216Metric" V 6530 4600 50  0001 C CNN
 F 3 "~" H 6600 4600 50  0001 C CNN
@@
 P 6850 4600
 F 0 "R24" H 6920 4646 50  0000 L CNN
-F 1 "R" H 6920 4555 50  0000 L CNN
+F 1 "4.7K" H 6920 4555 50  0000 L CNN
 F 2 "Resistor_SMD:R_1206_3216Metric" V 6780 4600 50  0001 C CNN
 F 3 "~" H 6850 4600 50  0001 C CNN
@@
 	5950 6700 5650 6700
 Connection ~ 5650 6700
+$Comp
+L Device:C C13
+U 1 1 5FDC513A
+P 6800 6900
+F 0 "C13" H 6915 6946 50  0000 L CNN
+F 1 ".1uF" H 6915 6855 50  0000 L CNN
+F 2 "Capacitor_SMD:C_1206_3216Metric" H 6838 6750 50  0001 C CNN
+F 3 "~" H 6800 6900 50  0001 C CNN
+	1    6800 6900
+	1    0    0    -1
+$EndComp
+Wire Wire Line
+	6650 6450 6800 6450
+Wire Wire Line
+	6800 6450 6800 6750
+Wire Wire Line
+	6500 6750 6500 7050
+Wire Wire Line
+	6500 7050 6800 7050
+Connection ~ 6500 6750
+Wire Wire Line
+	6500 6750 6350 6750
 $EndSCHEMATC
