File: herbie2/herbie2_pcb/herbie2.kicad_pcb (KiCad board)
At the start: 2 copper layers, 119.4 x 96.5 mm, 96 parts, among them J1 GND, J10 CONN_04JST-PTH, J11 CONN_04JST-PTH, J12 Vin, J15 Conn_01x03_Male, J16 Conn_02x03_Odd_Even, J17 Conn_01x03, J18 Conn_01x02, J19 Conn_01x01, J2 5V, J20 Conn_01x03, J3 I2C_STANDARDQWIIC, J4 Conn_01x01, J5 Conn_01x02, J8 I2C_STANDARDQWIIC, J9 I2C_STANDARDQWIIC, Q1 LTC4412, Q2 LTC4412, Q3 Si4427, Q4 Si4427, Q5 2N7002, U1 74HC595, U2 74164, U3 24v13_Pololu, U4 LS7366R, U5 LS7366R, U6 TCA9534, U7 24v13_Pololu, U8 D36V50F5_Pololu, Y1 20MHz, Y2 20MHz

Commit message: v0.1
Parts:
- added C13: .1uF, Capacitor_SMD:C_1206_3216Metric, F.Cu at (202.6, 99.7)
- R21, R22: value 47K -> 20K
- R23, R24: value R -> 4.7K
- RV1: value 1K -> 10K
- turned D1 to 90 degrees
- turned D3 to 90 degrees
Connections:
- D1 pad 1: GND -> Net-(D1-Pad1)
- D1 pad 2: Net-(D1-Pad2) -> 3.3V
- D2 pad 1: GND -> Net-(D2-Pad1)
- D2 pad 2: Net-(D2-Pad2) -> 3.3V
- D3 pad 1: GND -> Net-(D3-Pad1)
- D3 pad 2: Net-(D3-Pad2) -> 3.3V
- D4 pad 1: GND -> Net-(D4-Pad1)
- D4 pad 2: Net-(D4-Pad2) -> 3.3V
- R3 pad 2: Net-(D1-Pad2) -> Net-(D1-Pad1)
- R4 pad 2: Net-(D2-Pad2) -> Net-(D2-Pad1)
- R5 pad 2: Net-(D3-Pad2) -> Net-(D3-Pad1)
- R6 pad 2: Net-(D4-Pad2) -> Net-(D4-Pad1)
Routing:
- net 3.3V: track 319.2 -> 401.4 mm, vias 10 -> 12
- net Net-(D2-Pad1): track 0.00 -> 37.5 mm
- net Net-(D2-Pad2): track 34.5 -> 0.00 mm
- net GND: track 218.0 -> 197.8 mm, vias 24 -> 21
- net Net-(D3-Pad2): track 12.7 -> 0.00 mm
- net Net-(D3-Pad1): track 0.00 -> 11.7 mm
- net SCL: track 194.2 -> 182.6 mm, vias 7 -> 6
- net Net-(D4-Pad1): track 0.00 -> 6.27 mm
- net Net-(D4-Pad2): track 5.11 -> 0.00 mm
- net Net-(D1-Pad2): track 3.84 -> 0.00 mm
- net Net-(D1-Pad1): track 0.00 -> 3.84 mm
