File: herbie_nn/herbie2_pcb/vexu/magic_board/magic_board.kicad_sch (KiCad schematic)
At the start: 78 parts, among them J1 4P4C, J2 Conn_ARM_JTAG_SWD_10, J3 USB_C_Receptacle_USB2.0_14P, J4 Conn_01x04_Pin, J5 Conn_01x04_Pin, U11 74LVC125, U12 AMS1117-5.0, U13 AP2112K-3.3, U14 74LVC2G14, U15 74LVC125, U2 AT25SF081-SSHD-X, U3 LM386, U4 ATSAMD51J19A-A, U5 LS7366R, U6 LS7366R, U7 LS7366R, U8 LS7366R, Y1 32.768KHz, Y2 8MHz

Commit message: added labels and logo
Parts:
- removed C14: C, Capacitor_SMD:C_1206_3216Metric, symbol Device:C
- removed J4, J5: Conn_01x04_Pin, Connector_PinHeader_2.54mm:PinHeader_1x04_P2.54mm_Vertical, symbol Connector:Conn_01x04_Pin
- removed R18, R19, R8: R, Resistor_SMD:R_1206_3216Metric, symbol Device:R
- removed TP1: TestPoint, TestPoint:TestPoint_Pad_D1.0mm, symbol Connector:TestPoint
- removed U3: LM386, Package_SO:SOIC-8-1EP_3.9x4.9mm_P1.27mm_EP2.29x3mm, symbol Amplifier_Audio:LM386
- added C4: 1uF, Capacitor_SMD:C_1206_3216Metric, symbol Device:C
- added C5: 10uF, Capacitor_SMD:C_1206_3216Metric, symbol Device:C
- added J4: Conn_01x04_Socket, Connector_PinHeader_1.27mm:PinHeader_1x04_P1.27mm_Vertical, symbol Connector:Conn_01x04_Socket
- added J5, J6, J7: Conn_01x05_Pin, Connector_PinHeader_2.54mm:PinHeader_1x05_P2.54mm_Vertical, symbol Connector:Conn_01x05_Pin
- added L1: 10uH, Inductor_SMD:L_1206_3216Metric, symbol Device:L
- added Q2: MMBT3904, Package_TO_SOT_SMD:SOT-23, symbol Transistor_BJT:MMBT3904
- added R10, R13: R, Resistor_SMD:R_1206_3216Metric, symbol Device:R
- added R11, R9: 5.1K, Resistor_SMD:R_1206_3216Metric, symbol Device:R
- added R12: 1K, Resistor_SMD:R_1206_3216Metric, symbol Device:R
- added RESET1: SW_SPST, Button_Switch_SMD:SW_Push_1P1T_NO_CK_KMR2, symbol Switch:SW_SPST
- C10, C9: value C -> 12pF
- C11, C12, C3, C6: value C -> .1uF
- C13: value C -> 22uF
Connections:
- net +3.3V: now also C11.1, C12.1, U4.8 (VDDANA), J4.1 (Pin_1), J5.2 (Pin_2), R10.1
- net +5V: now also J5.1 (Pin_1), R13.1
- net BUZ_PIN: now also R12.1; no longer BZ1.1 (+)
- net DAC_OUT0: now also J5.4 (Pin_4)
- net DATA+: now also J1.2, R2.2; no longer J1.1, R1.2
- net DATA-: now also J1.1, R1.2; no longer J1.2, R2.2
- net GND: now also C11.2, C12.2, C13.2, ENC1.1 (Pin_1), ENC2.1 (Pin_1), ENC3.1 (Pin_1), ENC4.1 (Pin_1), C4.2, C5.2, J4.4 (Pin_4), J5.5 (Pin_5), J6.5 (Pin_5), J7.5 (Pin_5), Q2.2 (E), R11.2, R9.2, RESET1.1 (A); no longer BZ1.2 (-)
- net NRESET: now also R10.2, RESET1.2 (B)
- net SCL: now also J4.2 (Pin_2)
- net SDA: now also J4.3 (Pin_3)
- net SERCOM0.0: now also J6.1 (Pin_1)
- net SERCOM0.1: now also J6.2 (Pin_2)
- net SERCOM0.2: now also J6.3 (Pin_3)
- net SERCOM0.3: now also J6.4 (Pin_4)
- net SERCOM1.0: now also J7.1 (Pin_1)
- net SERCOM1.1: now also J7.2 (Pin_2)
- net SERCOM1.2: now also J7.3 (Pin_3)
- net SERCOM1.3: now also J7.4 (Pin_4)
- net at D3.2 (A), U12.2 (VO): now also C13.1
- net at J3.A5 (CC1): now also R9.1
- net at J3.B5 (CC2): now also R11.1
- net LED2_PIN: now reaches R5.2
- net LED2_PIN: now also U4.44 (PA23)
- net PA03: now reaches U4.4 (PA03)
- net LED1_PIN: now reaches U4.43 (PA22)
- net LED1_PIN: now also R4.2
- net at U4.53 (VDDCORE): now also C4.1, C5.1, L1.1
- net at U4.55 (VSW): now also L1.2
- new net: BZ1.1 (+), R13.2
- new net: Q2.1 (B), R12.2
- new net: BZ1.2 (-), Q2.3 (C)
- new net PA_03: J5.3 (Pin_3)
- no-connect marks 21 -> 23
Other:
- moved on the sheet: BZ1

Commit message: version 0.1 sent for fabrication
Parts:
- added F1: 500mA, Fuse:Fuse_1206_3216Metric, symbol Device:Fuse
- added R14: 1K, Resistor_SMD:R_1206_3216Metric, symbol Device:R
- added R8: 10K, Resistor_SMD:R_1206_3216Metric, symbol Device:R
- R10: value R -> 10K
- R20, R21, R22, R23, R24, R25, R26, R27: value R -> 100
Connections:
- net PA03 is gone; now on net PA_03: U4.4 (PA03)
- net +3.3V: now also R8.1
- net GND: now also J2.9 (GNDDetect)
- net QSPI_CS: now also R8.2
- net at BZ1.1 (+), R13.2: now also R14.2
- net at J3.A4 (VBUS), J3.A9 (VBUS), J3.B4 (VBUS)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: now also F1.1; no longer D2.2 (A)
- net at BZ1.2 (-), Q2.3 (C): now also R14.1
- new net: D2.2 (A), F1.2
- no-connect marks 23 -> 33
Other:
- moved on the sheet: BZ1, D2, R13
