File: herbie_nn/herbie2_pcb/vexu/magic_board/magic_board.kicad_pcb (KiCad board)
At the start: 2 copper layers, 70 x 50 mm, 92 parts, among them J1 4P4C, J2 Conn_ARM_JTAG_SWD_10, J3 USB_C_Receptacle_USB2.0_14P, J4 Conn_01x04_Socket, J5 Conn_01x05_Pin, J6 Conn_01x05_Pin, J7 Conn_01x05_Pin, J8 Conn_01x04_Socket, Q2 MMBT3904, U11 74LVC125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

Commit message: v0.2 pre1
Routing:
- net /SCL: track 36.7 -> 37.3 mm
Changed lines of the file:
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@@
 		(tags "resistor")
 		(property "Reference" "R16"
-			(at 0 1.82 0)
+			(at -1.4625 1.82 0)
 			(layer "B.SilkS")
 			(effects
@@
 		(tags "resistor")
 		(property "Reference" "R14"
-			(at 0 1.82 90)
+			(at 1.33 -2.22 90)
 			(layer "B.SilkS")
 			(effects
@@
 	)
 	(segment
-		(start 77 96.97)
-		(end 79.6 94.37)
-		(width 0.2)
-		(layer "F.Cu")
-		(net 3)
-	)
-	(segment
 		(start 75 104.75)
 		(end 75.0125 104.75)
@@
 	)
 	(segment
+		(start 78.8525 95.1175)
+		(end 79.6 94.37)
+		(width 0.2)
+		(layer "F.Cu")
+		(net 3)
+	)
+	(segment
 		(start 77 99.2)
 		(end 77.74 99.94)
@@
 	)
 	(segment
-		(start 77 99.2)
-		(end 77 96.97)
+		(start 77 98.485)
+		(end 78.8525 96.6325)
 		(width 0.2)
 		(layer "F.Cu")
@@
 	)
 	(segment
+		(start 78.8525 96.6325)
+		(end 78.8525 95.1175)
+		(width 0.2)
+		(layer "F.Cu")
+		(net 3)
+	)
+	(segment
+		(start 77 99.2)
+		(end 77 98.485)
+		(width 0.2)
+		(layer "F.Cu")
+		(net 3)
+	)
+	(segment
 		(start 75 106.25)
 		(end 75 110.35)
@@
 	)
 	(segment
-		(start 78.275 76.725)
-		(end 78.275 75.9)
-		(width 0.2)
+		(start 83.646 74.659754)
+		(end 84.059754 74.246)
+		(width 0.508)
+		(layer "F.Cu")
+		(net 78)
+	)
+	(segment
+		(start 78.075 75.9)
+		(end 78.075 76.925)
+		(width 0.508)
+		(layer "F.Cu")
+		(net 78)
+	)
+	(segment
+		(start 84.059754 74.246)
+		(end 84.219395 74.246)
+		(width 0.508)
 		(layer "F.Cu")
 		(net 78)
@@
 	)
 	(segment
-		(start 58.67 81.6975)
-		(end 58.67 80.48)
-		(width 0.1778)
+		(start 83.646 75.446)
+		(end 83.646 74.659754)
+		(width 0.508)
 		(layer "F.Cu")
 		(net 78)
 	)
 	(segment
-		(start 77.8 77.2)
-		(end 78.275 76.725)
-		(width 0.2)
+		(start 58.67 81.6975)
+		(end 58.67 80.48)
+		(width 0.1778)
 		(layer "F.Cu")
 		(net 78)
@@
 	)
 	(segment
-		(start 58.28 80.48)
-		(end 57.8 80)
-		(width 0.1778)
-		(layer "F.Cu")
-		(net 78)
-	)
-	(segment
-		(start 85.565395 72.9)
-		(end 84.219395 74.246)
+		(start 84.219395 74.246)
+		(end 85.565395 72.9)
 		(width 0.508)
 		(layer "F.Cu")
@@
 	)
 	(segment
-		(start 86.2 72.9)
-		(end 85.565395 72.9)
-		(width 0.508)
+		(start 58.28 80.48)
+		(end 57.8 80)
+		(width 0.1778)
 		(layer "F.Cu")
 		(net 78)
 	)
 	(segment
-		(start 83.4 74.905754)
-		(end 83.4 75.8)
+		(start 85.565395 72.9)
+		(end 86.2 72.9)
 		(width 0.508)
 		(layer "F.Cu")
@@
 	)
 	(segment
-		(start 84.059754 74.246)
-		(end 83.4 74.905754)
+		(start 84 75.8)
+		(end 83.646 75.446)
 		(width 0.508)
 		(layer "F.Cu")
@@
 	)
 	(segment
-		(start 84.219395 74.246)
-		(end 84.059754 74.246)
+		(start 78.075 76.925)
+		(end 77.8 77.2)
 		(width 0.508)
 		(layer "F.Cu")
@@
 	)
 	(via
-		(at 83.4 75.8)
+		(at 84 75.8)
 		(size 0.6)
 		(drill 0.3)
@@
 	)
 	(segment
-		(start 78.875 77.2)
-		(end 79.075 77)
-		(width 0.2)
-		(layer "B.Cu")
-		(net 78)
-	)
-	(segment
-		(start 80 77)
-		(end 79.075 77)
+		(start 84 75.8)
+		(end 81.2 75.8)
 		(width 0.2)
 		(layer "B.Cu")
@@
 	)
 	(segment
-		(start 77.8 77.2)
-		(end 78.875 77.2)
+		(start 81.2 75.8)
+		(end 80 77)
 		(width 0.2)
 		(layer "B.Cu")
@@
 	)
 	(segment
-		(start 83.4 75.8)
-		(end 81.2 75.8)
+		(start 78.875 77.2)
+		(end 79.075 77)
 		(width 0.2)
 		(layer "B.Cu")
@@
 	)
 	(segment
-		(start 81.2 75.8)
-		(end 80 77)
+		(start 77.8 77.2)
+		(end 78.875 77.2)
 		(width 0.2)
 		(layer "B.Cu")
@@
 		(layer "B.Cu")
 		(net 78)
+	)
+	(segment
+		(start 80 77)
+		(end 79.075 77)
+		(width 0.2)
+		(layer "B.Cu")
+		(net 78)

Commit message: Version 0.2 PCB
Routing:
- net +3.3V: track 296.1 -> 294.4 mm
Changed lines of the file:
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@@
-	)
-	(segment
-		(start 52.180218 81.62)
-		(end 52.100218 81.7)
-		(width 0.762)
-		(layer "F.Cu")
-		(net 13)
 	)
 	(segment
@@
 	)
 	(segment
-		(start 52.100218 81.7)
-		(end 51.475 81.7)
-		(width 0.762)
-		(layer "F.Cu")
-		(net 13)
-	)
-	(segment
 		(start 59.326069 91.11)
 		(end 58.716069 90.5)
@@
 		(layer "F.Cu")
 		(net 13)
-	)
-	(segment
-		(start 52.909 80.891218)
-		(end 52.180218 81.62)
-		(width 0.508)
-		(layer "F.Cu")
-		(net 13)
