File: astromech/Dome/Dome_Board/Dome_Board/Dome_Board.kicad_sch (KiCad schematic)
At the start: 12 parts, among them J1 Conn_01x02_Socket, J10 Conn_01x02_Socket, J2 Conn_01x02_Socket, J3 Conn_01x02_Socket, J4 Conn_01x03_Pin, J5 Conn_01x03_Pin, J6 Conn_01x03_Pin, J7 Conn_01x03_Pin, J8 Conn_01x03_Pin, J9 Conn_01x03_Pin, U1 ESP32-C6-DEVKITC-1-N8, U3 D36V50F5_Pololu

Commit message: added more PWM and Servo driver
Parts:
- removed J4, J5, J6, J7, J8, J9: Conn_01x03_Pin, Connector_PinHeader_2.54mm:PinHeader_1x03_P2.54mm_Vertical, symbol Connector:Conn_01x03_Pin
- added C1: C, Capacitor_SMD:C_1206_3216Metric_Pad1.33x1.80mm_HandSolder, symbol Device:C
- added J26: Conn_01x23_Pin, Connector_PinHeader_2.54mm:PinHeader_1x23_P2.54mm_Vertical, symbol Connector:Conn_01x23_Pin
- added Q1, Q2: BSS138, Package_TO_SOT_SMD:SOT-23, symbol Transistor_FET:BSS138
- added R1, R10, R11, R12, R13, R14, R15, R16, R17, R18, R19, R2, R20, R21, R22, R23, R24, R25, R3, R4, R5, R6, R7, R8, R9: R, Resistor_SMD:R_1206_3216Metric_Pad1.30x1.75mm_HandSolder, symbol Device:R
- added U2: PCA9685PW, custom_library:SOT361-1_NXP-M, symbol custom_library:PCA9685PW
Connections:
- net +5V: now also C1.2, J26.1 (Pin_1), R23.1, R25.1, U2.28 (VDD)
- net GND: now also C1.1, J26.23 (Pin_23), U2.14 (VSS)
- net PWM 1: now also U1.J3_4 (GPIO15), R1.1; no longer U1.J3_5 (GPIO23)
- net PWM 2: now also U1.J3_5 (GPIO23), R2.1; no longer U1.J3_6 (GPIO22)
- net PWM 3: now also U1.J3_6 (GPIO22), R3.1; no longer U1.J3_7 (GPIO21)
- net PWM 4: now also U1.J3_7 (GPIO21), R4.1; no longer U1.J3_8 (GPIO20)
- net PWM 5: now also U1.J3_8 (GPIO20), R5.1; no longer U1.J3_9 (GPIO19)
- net PWM 6: now also R6.1, U2.6 (LED0); no longer U1.J3_10 (GPIO18)
- net scl: now also Q2.2 (S), R24.2
- net sda: now also Q1.2 (S), R22.2
- net 3V3: now reaches U1.J1_1 (ESP_3V3)
- net 3V3: now also Q1.1 (G), Q2.1 (G), R22.1, R24.1
- new net: J26.22 (Pin_22), R21.2
- new net: J26.15 (Pin_15), R14.2
- new net: J26.10 (Pin_10), R9.2
- new net: J26.9 (Pin_9), R8.2
- new net: J26.8 (Pin_8), R7.2
- new net: J26.3 (Pin_3), R2.2
- new net: J26.11 (Pin_11), R10.2
- new net: J26.12 (Pin_12), R11.2
- new net: J26.13 (Pin_13), R12.2
- new net: J26.14 (Pin_14), R13.2
- new net: J26.16 (Pin_16), R15.2
- new net: J26.17 (Pin_17), R16.2
- new net: J26.18 (Pin_18), R17.2
- new net: J26.19 (Pin_19), R18.2
- new net: J26.2 (Pin_2), R1.2
- new net: J26.20 (Pin_20), R19.2
- new net: J26.21 (Pin_21), R20.2
- new net: J26.4 (Pin_4), R3.2
- new net: J26.5 (Pin_5), R4.2
- new net: J26.6 (Pin_6), R5.2
- new net: J26.7 (Pin_7), R6.2
- new net PWM 10: R10.1, U2.10 (LED4)
- new net PWM 11: R11.1, U2.11 (LED5)
- new net PWM 12: R12.1, U2.12 (LED6)
- new net PWM 13: R13.1, U2.13 (LED7)
- new net PWM 14: R14.1, U2.15 (LED8)
- new net PWM 15: R15.1, U2.16 (LED9)
- new net PWM 16: R16.1, U2.17 (LED10)
- new net PWM 17: R17.1, U2.18 (LED11)
- new net PWM 18: R18.1, U2.19 (LED12)
- new net PWM 19: R19.1, U2.20 (LED13)
- new net PWM 20: R20.1, U2.21 (LED14)
- new net PWM 21: R21.1, U2.22 (LED15)
- new net PWM 7: R7.1, U2.7 (LED1)
- new net PWM 8: R8.1, U2.8 (LED2)
- new net PWM 9: R9.1, U2.9 (LED3)
- new net level converter magic: Q1.3 (D), R23.2, U2.27 (SDA)
- new net more level converter magic: Q2.3 (D), R25.2, U2.26 (SCL)

Commit message: added reset button
Parts:
- added C2: NC/100nF, Capacitor_SMD:C_1206_3216Metric_Pad1.33x1.80mm_HandSolder, symbol Device:C
- added SW1: COM-12992, custom_library:COM-12992_SPK, symbol 2024-11-02_20-09-58:COM-12992
Connections:
- net GND: now also C2.1, SW1.2
- net rst_button: now reaches U1.J1_2 (CHIP_PU)
- net rst_button: now also C2.2, SW1.4
- net level converter magic renamed SDA +5V
- net more level converter magic renamed SCL +5V
Other:
- moved on the sheet: J1, J10
